File: AS3310-ADSR.kicad_pcb (KiCad board)
At the start: 2 copper layers, 59 parts, among them J1 TRIGGER_IN, J2 EURO_PWR_2x5, J3 TRIGGER_IN, J4 TRIGGER_IN, Q1 BC558, Q2 BC548, SW2 SW_Push, U1 LM358, U2 AS3310, U3 LM358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

Commit message: Refactor
Parts:
- J3: value TRIGGER_IN -> ENVELOPE_OUT; footprint Seattle_Synths:Jack_3.5mm_QingPu_WQP-PJ398SM_Vertical_CircularHoles -> Seattle_Synths:CUI_MJ-63052A
- J4: value TRIGGER_IN -> GATE_IN
- moved S1 62.2 mm to (114.1, 144.0)
- moved J3 15.2 mm to (104.9, 73.9)
Other:
- board outline added: 2.1 x 2.1 mm

Commit message: Refacctor
Parts:
- added BOTTOM_LEFT_MOUNT: MountingHole_3.2mm_M3_Oval, Seattle_Synths:MountingHole_3.2mm_M3_Oval, F.Cu at (88.3, 163.0)
- added BOTTOM_RIGHT_MOUNT: MountingHole_3.2mm_M3_Oval, Seattle_Synths:MountingHole_3.2mm_M3_Oval, F.Cu at (144.8, 163.1)
- added D3: LED, Seattle_Synths:LED_D5.0mm, B.Cu at (142.6, 43.4)
- added R26: 330R, Seattle_Synths:R_Axial_DIN0207_L6.3mm_D2.5mm_P10.16mm_Horizontal, F.Cu at (139.4, 156.1)
- added TOP_LEFT_MOUNT: MountingHole_3.2mm_M3_Oval, Seattle_Synths:MountingHole_3.2mm_M3_Oval, F.Cu at (88.1, 35.7)
- added TOP_RIGHT_MOUNT: MountingHole_3.2mm_M3_Oval, Seattle_Synths:MountingHole_3.2mm_M3_Oval, F.Cu at (144.9, 35.7)
- added TP4: -12V, Seattle_Synths:TestPoint_Pad_4.0x4.0mm, F.Cu at (111.0, 37.1)
- added TP5: GND, Seattle_Synths:TestPoint_Pad_4.0x4.0mm, F.Cu at (117.5, 37.0)
- added TP6: +12V, Seattle_Synths:TestPoint_Pad_4.0x4.0mm, F.Cu at (123.7, 37.0)
- J1, J4, RV1, RV2, RV3, RV4, S1, SW2: moved to B.Cu
- J2: value EURO_PWR_2x5 -> -----
- J3: footprint Seattle_Synths:CUI_MJ-63052A -> Seattle_Synths:Jack_3.5mm_QingPu_WQP-PJ398SM_Vertical_CircularHoles; moved to B.Cu
- moved RV6 104.1 mm to (88.2, 42.2)
- moved RV4 97.9 mm to (131.2, 78.6), turned to 90 degrees
- moved U1 87.4 mm to (102.5, 149.9)
- moved U3 85.6 mm to (116.5, 136.0)
- moved R12 84.2 mm to (84.8, 155.8)
- moved C4 84.0 mm to (129.7, 157.1)
- moved RV3 83.2 mm to (131.5, 53.5), turned to 90 degrees
- moved R7 82.7 mm to (85.3, 129.9)
- moved TP3 81.5 mm to (124.3, 151.3)
- moved R5 79.0 mm to (85.4, 119.4)
- moved TP2 77.7 mm to (120.0, 160.0)
- moved D2 75.1 mm to (121.8, 61.1)
- moved C6 72.5 mm to (87.8, 91.4)
- moved C5 67.0 mm to (87.8, 84.4)
- moved D1 66.3 mm to (108.4, 61.0)
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Routing:
- net GND: track 0.00 -> 418.8 mm
- net +12V: track 0.00 -> 309.9 mm
- net -12V: track 0.00 -> 214.4 mm, vias 0 -> 1
- net /OUT2: track 0.00 -> 181.9 mm
- net /GATE: track 0.00 -> 165.5 mm
- net /TRIG: track 0.00 -> 138.6 mm
- net /RELEASE: track 0.00 -> 128.7 mm
- net /ENVOUT: track 0.00 -> 125.4 mm
- net Net-(C6-Pad2): track 0.00 -> 123.1 mm
- net Net-(C5-Pad1): track 0.00 -> 122.5 mm, vias 0 -> 1
- net Net-(D3-Pad2): track 0.00 -> 119.1 mm
- net Net-(J4-PadTN): track 0.00 -> 108.5 mm
- net /SUSTAIN: track 0.00 -> 98.8 mm
- net Net-(R3-Pad2): track 0.00 -> 97.2 mm
- net /OUT4: track 0.00 -> 94.9 mm
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Other:
- board size 2.1 x 2.1 mm -> 71 x 133.1 mm
- board text added: "Seattle Synths SS-ADSR-1 Rev. 1 [2020-11-08]"
- board text added: "This machine kills fascists."

Commit message: Refactor
Parts:
- C10, C9: footprint Seattle_Synths:C_Disc_D7.5mm_W2.5mm_P5.00mm -> Seattle_Synths:CP_Radial_D5.0mm_P2.50mm
- J2: value ----- -> EURO_PWR_2x5
- RV5, RV6: footprint Seattle_Synths:Potentiometer_Runtron_RM-065_Vertical -> Seattle_Synths:TRIM_3266W-1-102LF
- moved C9 65.0 mm to (97.1, 86.3)
- moved C7 59.5 mm to (129.5, 142.6)
- moved RV6 5.01 mm to (89.7, 47.0)
- moved RV5 4.56 mm to (117.0, 117.0)
- moved C10 4.55 mm to (103.6, 86.3)
- moved Q1 0.82 mm to (129.4, 103.3)
- moved Q2 0.55 mm to (129.4, 111.3)
Routing:
- net /OUT2: track 181.9 -> 133.1 mm
- net Net-(R3-Pad2): track 97.2 -> 56.1 mm
- net -12V: track 214.4 -> 254.6 mm, vias 1 -> 0
- net /IIN: track 43.5 -> 69.7 mm
- net Net-(RV1-Pad2): track 36.7 -> 59.3 mm
- net /GATE: track 165.5 -> 143.6 mm
- net /TRIG: track 138.6 -> 118.8 mm
- net +12V: track 309.9 -> 291.5 mm, vias 0 -> 1
- net GND: track 418.8 -> 436.7 mm
- net Net-(C7-Pad2): track 53.2 -> 37.3 mm, vias 1 -> 0
- net Net-(C1-Pad1): track 81.8 -> 69.7 mm
- net /OUT4: track 94.9 -> 104.9 mm
- net /IN1: track 76.7 -> 86.1 mm
- net /ENVOUT: track 125.4 -> 117.0 mm
- net Net-(C6-Pad2): track 123.1 -> 115.5 mm, vias 0 -> 1
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
Commit message: Refactor
Parts:
- SW2: footprint Seattle_Synths:SW_PUSH_6mm_H5mm -> Seattle_Synths:SW_PS1024ALRED
- moved SW2 5.09 mm to (143.3, 75.2)
- moved J2 1.90 mm to (143.1, 53.0)
Routing:
- net /IIN: track 69.7 -> 45.7 mm
- net Net-(RV1-Pad2): track 59.3 -> 42.0 mm, vias 0 -> 1
- net -12V: track 254.6 -> 271.4 mm, vias 0 -> 1
- net Net-(J4-PadTN): track 113.8 -> 98.6 mm
- net /OUT4: track 104.9 -> 92.1 mm
- net /RELEASE: track 134.8 -> 143.8 mm
- net +12V: track 291.5 -> 285.0 mm
- net GND: track 436.7 -> 432.1 mm
- net Net-(D3-Pad2): track 124.1 -> 119.8 mm
- net Net-(R3-Pad2): track 56.1 -> 52.5 mm
- net Net-(R2-Pad2): track 68.0 -> 65.5 mm
- net /IN1: track 86.1 -> 84.5 mm
- net /IN2: track 32.4 -> 31.2 mm
- net Net-(J3-PadT): track 79.0 -> 79.9 mm
- net Net-(C6-Pad2): track 115.5 -> 116.3 mm
